File: examples/air_quality_sensor/air_quality_sensor.kicad_pcb (KiCad board)
At the start: 2 copper layers, 0 parts

Commit message: fix: extract _impl_* helpers in routing.py to fix autoroute FunctionTool bug
The autoroute tool was crashing with TypeError because it called
clean_board_for_routing, export_dsn, run_freerouter, and import_ses as
plain functions — but @mcp.tool() decoration makes them FunctionTool
objects, not callables.

Fix: extracted the body of each routing tool into module-level _impl_*
helper functions. The @mcp.tool() wrappers delegate to the helpers;
autoroute calls the helpers directly, bypassing the FunctionTool layer.

Also:
- Added stdin=subprocess.DEVNULL to FreeRouting subprocess call to
  prevent blocking on the MCP stdio pipe
- Fixed test_run_freerouter to use the real DSN from test_export_dsn
  instead of a dummy file (dummy DSN always fails FreeRouting validation)
- Updated LESSONS_LEARNED.md with lessons 24-26

Result: 63/64 pass, 1 skip (run_freerouter skipped when pcbnew
unavailable so export_dsn cannot produce a valid DSN), 0 fail.

Co-Authored-By: Claude Sonnet 4.6 <noreply@anthropic.com>
Parts:
- added C1: , Capacitor_SMD:C_0402_1005Metric, F.Cu at (50.0, 50.0)
- added C2: , Capacitor_SMD:C_0402_1005Metric, F.Cu at (60.0, 50.0)
- added C3: , Capacitor_SMD:C_0402_1005Metric, F.Cu at (70.0, 50.0)
- added C4: , Capacitor_SMD:C_0402_1005Metric, F.Cu at (80.0, 50.0)
- added C5: , Capacitor_SMD:C_0402_1005Metric, F.Cu at (90.0, 50.0)
- added C6: , Capacitor_SMD:C_0402_1005Metric, F.Cu at (100.0, 50.0)
- added J1: , Connector_PinHeader_2.54mm:PinHeader_1x02_P2.54mm_Vertical, F.Cu at (110.0, 50.0)
- added J2: , Connector_PinHeader_2.54mm:PinHeader_1x04_P2.54mm_Vertical, F.Cu at (120.0, 50.0)
- added R1: , Resistor_SMD:R_0402_1005Metric, F.Cu at (130.0, 50.0)
- added R2: , Resistor_SMD:R_0402_1005Metric, F.Cu at (140.0, 50.0)
- added U1: , Package_SO:SOIC-8_3.9x4.9mm_P1.27mm, F.Cu at (150.0, 50.0)
- added U2: , Package_DFN_QFN:DFN-10_3x3mm_P0.5mm, F.Cu at (160.0, 50.0)
- added U3: , Package_DFN_QFN:DFN-6_3x3mm_P1mm_PullbackPads0.25mm_BackPad, F.Cu at (170.0, 50.0)
- added U4: , Package_TO_SOT_SMD:SOT-223-3_TabPin2, F.Cu at (180.0, 50.0)
Changed lines of the file:
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@@
   (net 4 "SDA")
   (net 5 "SCL")
+  (footprint "Capacitor_SMD:C_0402_1005Metric" (layer "F.Cu")
+    (at 50.0 50.0)
+    (property "Reference" "C1" (at 0 0 0)
+      (effects (font (size 1 1) (thickness 0.15)))
+    )
+    (property "Value" "" (at 0 0 0)
+      (effects (font (size 1 1) (thickness 0.15)))
+    )
+  )
+  (footprint "Capacitor_SMD:C_0402_1005Metric" (layer "F.Cu")
+    (at 60.0 50.0)
+    (property "Reference" "C2" (at 0 0 0)
+      (effects (font (size 1 1) (thickness 0.15)))
+    )
+    (property "Value" "" (at 0 0 0)
+      (effects (font (size 1 1) (thickness 0.15)))
+    )
+  )
+  (footprint "Capacitor_SMD:C_0402_1005Metric" (layer "F.Cu")
+    (at 70.0 50.0)
+    (property "Reference" "C3" (at 0 0 0)
+      (effects (font (size 1 1) (thickness 0.15)))
+    )
+    (property "Value" "" (at 0 0 0)
+      (effects (font (size 1 1) (thickness 0.15)))
+    )
+  )
+  (footprint "Capacitor_SMD:C_0402_1005Metric" (layer "F.Cu")
+    (at 80.0 50.0)
+    (property "Reference" "C4" (at 0 0 0)
+      (effects (font (size 1 1) (thickness 0.15)))
+    )
+    (property "Value" "" (at 0 0 0)
+      (effects (font (size 1 1) (thickness 0.15)))
+    )
+  )
+  (footprint "Capacitor_SMD:C_0402_1005Metric" (layer "F.Cu")
+    (at 90.0 50.0)
+    (property "Reference" "C5" (at 0 0 0)
+      (effects (font (size 1 1) (thickness 0.15)))
+    )
+    (property "Value" "" (at 0 0 0)
+      (effects (font (size 1 1) (thickness 0.15)))
+    )
+  )
+  (footprint "Capacitor_SMD:C_0402_1005Metric" (layer "F.Cu")
+    (at 100.0 50.0)
+    (property "Reference" "C6" (at 0 0 0)
+      (effects (font (size 1 1) (thickness 0.15)))
+    )
+    (property "Value" "" (at 0 0 0)
+      (effects (font (size 1 1) (thickness 0.15)))
+    )
+  )
+  (footprint "Connector_PinHeader_2.54mm:PinHeader_1x02_P2.54mm_Vertical" (layer "F.Cu")
+    (at 110.0 50.0)
+    (property "Reference" "J1" (at 0 0 0)
+      (effects (font (size 1 1) (thickness 0.15)))
+    )
+    (property "Value" "" (at 0 0 0)
+      (effects (font (size 1 1) (thickness 0.15)))
+    )
+  )
+  (footprint "Connector_PinHeader_2.54mm:PinHeader_1x04_P2.54mm_Vertical" (layer "F.Cu")
+    (at 120.0 50.0)
+    (property "Reference" "J2" (at 0 0 0)
+      (effects (font (size 1 1) (thickness 0.15)))
+    )
+    (property "Value" "" (at 0 0 0)
+      (effects (font (size 1 1) (thickness 0.15)))
+    )
+  )
+  (footprint "Resistor_SMD:R_0402_1005Metric" (layer "F.Cu")
+    (at 130.0 50.0)
+    (property "Reference" "R1" (at 0 0 0)
+      (effects (font (size 1 1) (thickness 0.15)))
+    )
+    (property "Value" "" (at 0 0 0)
+      (effects (font (size 1 1) (thickness 0.15)))
+    )
+  )
+  (footprint "Resistor_SMD:R_0402_1005Metric" (layer "F.Cu")
+    (at 140.0 50.0)
+    (property "Reference" "R2" (at 0 0 0)
+      (effects (font (size 1 1) (thickness 0.15)))
+    )
+    (property "Value" "" (at 0 0 0)
+      (effects (font (size 1 1) (thickness 0.15)))
+    )
+  )
+  (footprint "Package_SO:SOIC-8_3.9x4.9mm_P1.27mm" (layer "F.Cu")
+    (at 150.0 50.0)
+    (property "Reference" "U1" (at 0 0 0)
+      (effects (font (size 1 1) (thickness 0.15)))
+    )
+    (property "Value" "" (at 0 0 0)
+      (effects (font (size 1 1) (thickness 0.15)))
+    )
+  )
+  (footprint "Package_DFN_QFN:DFN-10_3x3mm_P0.5mm" (layer "F.Cu")
+    (at 160.0 50.0)
+    (property "Reference" "U2" (at 0 0 0)
+      (effects (font (size 1 1) (thickness 0.15)))
+    )
+    (property "Value" "" (at 0 0 0)
+      (effects (font (size 1 1) (thickness 0.15)))
+    )
+  )
+  (footprint "Package_DFN_QFN:DFN-6_3x3mm_P1mm_PullbackPads0.25mm_BackPad" (layer "F.Cu")
+    (at 170.0 50.0)
+    (property "Reference" "U3" (at 0 0 0)
+      (effects (font (size 1 1) (thickness 0.15)))
+    )
+    (property "Value" "" (at 0 0 0)
+      (effects (font (size 1 1) (thickness 0.15)))
+    )
+  )
+  (footprint "Package_TO_SOT_SMD:SOT-223-3_TabPin2" (layer "F.Cu")
+    (at 180.0 50.0)
+    (property "Reference" "U4" (at 0 0 0)
+      (effects (font (size 1 1) (thickness 0.15)))
+    )
+    (property "Value" "" (at 0 0 0)
+      (effects (font (size 1 1) (thickness 0.15)))
+    )
+  )
 )
