File: examples/air_quality_sensor/air_quality_sensor.kicad_sch (KiCad schematic)
At the start: 14 parts, among them J1 Conn_01x02, J2 Conn_01x04, U1 ATtiny85-20S, U2 SCD41, U3 SGP41, U4 AMS1117-3.3

Commit message: fix: extract _impl_* helpers in routing.py to fix autoroute FunctionTool bug
The autoroute tool was crashing with TypeError because it called
clean_board_for_routing, export_dsn, run_freerouter, and import_ses as
plain functions — but @mcp.tool() decoration makes them FunctionTool
objects, not callables.

Fix: extracted the body of each routing tool into module-level _impl_*
helper functions. The @mcp.tool() wrappers delegate to the helpers;
autoroute calls the helpers directly, bypassing the FunctionTool layer.

Also:
- Added stdin=subprocess.DEVNULL to FreeRouting subprocess call to
  prevent blocking on the MCP stdio pipe
- Fixed test_run_freerouter to use the real DSN from test_export_dsn
  instead of a dummy file (dummy DSN always fails FreeRouting validation)
- Updated LESSONS_LEARNED.md with lessons 24-26

Result: 63/64 pass, 1 skip (run_freerouter skipped when pcbnew
unavailable so export_dsn cannot produce a valid DSN), 0 fail.

Co-Authored-By: Claude Sonnet 4.6 <noreply@anthropic.com>
Parts:
- C1, C2, C3, C4, C5, C6: footprint (none) -> Capacitor_SMD:C_0402_1005Metric
- J1: footprint (none) -> Connector_PinHeader_2.54mm:PinHeader_1x02_P2.54mm_Vertical
- J2: footprint (none) -> Connector_PinHeader_2.54mm:PinHeader_1x04_P2.54mm_Vertical
- R1, R2: footprint (none) -> Resistor_SMD:R_0402_1005Metric
- U1: footprint (none) -> Package_SO:SOIC-8_3.9x4.9mm_P1.27mm
- U2: footprint (none) -> Package_DFN_QFN:DFN-10_3x3mm_P0.5mm
- U3: footprint (none) -> Package_DFN_QFN:DFN-6_3x3mm_P1mm_PullbackPads0.25mm_BackPad
- U4: footprint (none) -> Package_TO_SOT_SMD:SOT-223-3_TabPin2
