File: tests/fixtures/sample_board.kicad_pcb (KiCad board)
At the start: 2 copper layers, 3 parts, among them U1 ATtiny85

Commit message: feat: harden IPC backend with file fallbacks, add create_project tool
All IPC operations now catch exceptions and fall back to the file
backend, so the MCP works correctly without a running KiCad instance.

Key changes:
- ipc_backend: IPCBoardOps, IPCSchematicOps, IPCLibraryOps all wrap
  IPC calls in try/except and delegate to FileBoardOps /
  FileSchematicOps / FileLibraryOps on any failure or timeout
- ipc_backend: _try_save_to_disk() catches ALL exceptions (was only
  catching RuntimeError), preventing cascade timeouts
- file_backend: implement FileSchematicOps.annotate() using regex-based
  reference designator assignment; add FileBoardOps.create_board()
- tools/project: add create_project tool (creates .kicad_pro,
  .kicad_sch, .kicad_pcb); uses KiCad installed template for .pro file
- tools/schematic: sync_schematic_to_pcb uses try-backend-first pattern
  so it degrades gracefully when IPC is unavailable
- platform_helper: add find_kicad_template_dir() for all platforms
- composite: add get_board_modify_ops() delegation
- tests: 204 pass, 1 skipped
Connections:
- R1 pad 1: VCC -> Net-(R1-1)
- R1 pad 2: SDA -> Net-(R1-2)
- R2 pad 1: VCC -> Net-(R2-1)
- R2 pad 2: SCL -> Net-(R2-2)
Changed lines of the file:
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@@
   (net 3 "SDA")
   (net 4 "SCL")
-  (footprint "Resistor_SMD:R_0805_2012Metric" (layer "F.Cu")
+    (net 5 "Net-(R1-1)")
+  (net 6 "Net-(R1-2)")
+  (net 7 "Net-(R2-1)")
+  (net 8 "Net-(R2-2)")
+(footprint "Resistor_SMD:R_0805_2012Metric" (layer "F.Cu")
     (at 100 50)
     (property "Reference" "R1")
     (property "Value" "10k")
-    (pad "1" smd roundrect (at -0.9125 0) (size 1 1.45) (layers "F.Cu" "F.Paste" "F.Mask") (net 1 "VCC"))
-    (pad "2" smd roundrect (at 0.9125 0) (size 1 1.45) (layers "F.Cu" "F.Paste" "F.Mask") (net 3 "SDA"))
+    (pad "1" smd roundrect (at -0.9125 0) (size 1 1.45) (layers "F.Cu" "F.Paste" "F.Mask") (net 5 "Net-(R1-1)"))
+    (pad "2" smd roundrect (at 0.9125 0) (size 1 1.45) (layers "F.Cu" "F.Paste" "F.Mask") (net 6 "Net-(R1-2)"))
   )
   (footprint "Resistor_SMD:R_0805_2012Metric" (layer "F.Cu")
@@
     (property "Reference" "R2")
     (property "Value" "4.7k")
-    (pad "1" smd roundrect (at -0.9125 0) (size 1 1.45) (layers "F.Cu" "F.Paste" "F.Mask") (net 1 "VCC"))
-    (pad "2" smd roundrect (at 0.9125 0) (size 1 1.45) (layers "F.Cu" "F.Paste" "F.Mask") (net 4 "SCL"))
+    (pad "1" smd roundrect (at -0.9125 0) (size 1 1.45) (layers "F.Cu" "F.Paste" "F.Mask") (net 7 "Net-(R2-1)"))
+    (pad "2" smd roundrect (at 0.9125 0) (size 1 1.45) (layers "F.Cu" "F.Paste" "F.Mask") (net 8 "Net-(R2-2)"))
   )
   (footprint "Package_SO:SOIC-8_3.9x4.9mm_P1.27mm" (layer "F.Cu")
